File: redtop_GST10.kicad_pcb (KiCad board)
At the start: 2 copper layers, 64.8 x 21.5 mm, 16 parts, among them J1 Conn_01x03, J2 Conn_01x05, U1 TLV274IN, U2 CD4013BE

Commit message: finalize r1 silkscreen
Parts:
- added REF**: OSHW-Logo_5.7x6mm_SilkScreen, Symbol:OSHW-Logo_5.7x6mm_SilkScreen, B.Cu at (139.8, 112.9)
- added REF**: KiCad-Logo2_5mm_SilkScreen, Symbol:KiCad-Logo2_5mm_SilkScreen, B.Cu at (94.6, 123.1)
Other:
- board text added: "by: JS"
